File: hardware/sheets/usb3-hub-A.kicad_sch (KiCad schematic)
At the start: 28 parts, among them U1 USB5744/2G, Y1 25MHz CL=20pF

Commit message: docs: C24 brain + bay cards — decisions, architecture, BOM card table, fabrication, README, USAGE, STATUS, changelog, history; diagrams: 8 slots, lid plan, left wall
Co-Authored-By: Claude Fable 5.1 <noreply@anthropic.com>
Parts:
- C161: renamed from R100; value 12.0k 1% -> 100n; footprint Resistor_SMD:R_0402_1005Metric -> Capacitor_SMD:C_0402_1005Metric; symbol Device:R -> Device:C
- C162: renamed from R101; value 10k -> 100n; footprint Resistor_SMD:R_0402_1005Metric -> Capacitor_SMD:C_0402_1005Metric; symbol Device:R -> Device:C
- C163: renamed from R102; value 10k -> 100n; footprint Resistor_SMD:R_0402_1005Metric -> Capacitor_SMD:C_0402_1005Metric; symbol Device:R -> Device:C
- C164: renamed from R103; value 200k -> 100n; footprint Resistor_SMD:R_0402_1005Metric -> Capacitor_SMD:C_0402_1005Metric; symbol Device:R -> Device:C
- R100: renamed from R113; value 10k -> 12.0k 1%
- R103: renamed from R124; value 10k -> 200k
- renumbered C161 to C153, C162 to C154, R114 to R101, R123 to R102
Connections:
- net +3V3: no longer C162.1, C163.1, R100.1, R103.1
- net BAY1_USB3_RX_N: now also C161.2; no longer C153.2
- net BAY2_USB3_RX_N: now also C162.2; no longer C154.2
- net GND: now also R100.2, R103.2; no longer C161.2, C164.2
- net U1_CFG_NON_REM: now also R103.1; no longer C164.1
- net U1_DN1_TXDM: now also C161.1; no longer C153.1
- net U1_DN2_TXDM: now also C162.1; no longer C154.1
- net U1_RBIAS: now also R100.1; no longer C161.1
- net U1_RESET_N: now also R102.2; no longer C163.2
- net U1_VBUS_DET: now also R101.2; no longer C162.2
- net U1_DN3_TXDP: now reaches U1.19 (USB3DN_TXDP3)
- net U1_DN3_TXDP: now also C153.1
- net U1_DN3_TXDM: now reaches U1.20 (USB3DN_TXDM3)
- net U1_DN3_TXDM: now also C163.1
- net BAY3_USB3_TX_P: now reaches U1.22 (USB3DN_RXDP3)
- net BAY3_USB3_TX_N: now reaches U1.23 (USB3DN_RXDM3)
- net U1_DN4_TXDP: now reaches U1.26 (USB3DN_TXDP4)
- net U1_DN4_TXDP: now also C154.1
- net U1_DN4_TXDM: now reaches U1.27 (USB3DN_TXDM4)
- net U1_DN4_TXDM: now also C164.1
- net BAY4_USB3_TX_P: now reaches U1.29 (USB3DN_RXDP4)
- net BAY4_USB3_TX_N: now reaches U1.30 (USB3DN_RXDM4)
- net U1_PRT_DIS_M3 renamed BAY3_USB2_DM
- net BAY3_USB2_DM: no longer R102.2
- net U1_PRT_DIS_M4 renamed BAY4_USB2_DM
- net BAY4_USB2_DM: no longer R103.2
- net U1_PRT_DIS_P3 renamed BAY3_USB2_DP
- net BAY3_USB2_DP: no longer R100.2
- net U1_PRT_DIS_P4 renamed BAY4_USB2_DP
- net BAY4_USB2_DP: no longer R101.2
- new net BAY3_USB3_RX_N: C163.2
- new net BAY3_USB3_RX_P: C153.2
- new net BAY4_USB3_RX_N: C164.2
- new net BAY4_USB3_RX_P: C154.2
- no-connect marks 15 -> 7
Other:
- note added: "Hub A: upstream on CM5 USB3-0. Downstream ports 1-4 -> bay slots 1-4 (C24: eight slots, four cards populated in v1)."
- note added: "usb3-hub-A: USB5744 hub A on CM5 USB3-0, bay slots 1-4"
- note removed: "Hub A: upstream on CM5 USB3-0. Downstream ports 1,2 -> bays 1,2. Ports 3,4 disabled by PRT_DIS straps (verify the strap resistor value against USB5744 §3.4.2)."
- note removed: "usb3-hub-A: USB5744 hub A on CM5 USB3-0, bays 1 and 2"
